Commit message: Clone of URDF without pot

File: iiwa_description/urdf/iiwa14_changed.xacro (robot description, xacro)
@@ -357,32 +357,4 @@
       </inertial>
     </link>
-    <joint name="iiwa_joint_pot" type="fixed">
-      <parent link="iiwa_link_ee"/>
-      <child link="iiwa_link_pot"/>
-      <!-- <origin rpy="0 0 0" xyz="0.015 -0.02 0.16"/> HIGHLY TUNED-->
-      <origin rpy="0 0 0" xyz="-0.01 -0.01 0.16"/>
-      <!-- <origin rpy="0 1.570796 0" xyz="0.095 0 0.15"/> -->
-    </joint>
-    <link name="iiwa_link_pot">
-      <inertial>
-        <origin rpy="0 1.57 0" xyz="0 0 0"/>
-        <mass value="0.0"/>
-        <inertia ixx="1" ixy="0" ixz="0" iyy="1" iyz="0" izz="1"/>
-      </inertial>
-      <visual>
-        <origin rpy="0 1.57 0" xyz="0 0 0"/>
-        <geometry>
-          <cylinder radius="0.1524" length="0.3556"/>
-        </geometry>
-        <material name="Grey"/>
-      </visual>
-      <collision>
-        <origin rpy="0 1.57 0" xyz="0 0 0"/>
-        <geometry>
-          <cylinder radius="0.1524" length="0.3556"/>
-        </geometry>
-        <material name="Grey"/>
-      </collision>
-    </link>
     <!--Extensions -->
     <xacro:iiwa_gazebo robot_name="${robot_name}" />
