Commit message: testing zero torque gazebo

File: iiwa_description/urdf/iiwa14-1.xacro (robot description, xacro)
@@ -60,5 +60,5 @@
   <xacro:property name="max_velocity_7" value="${135 * PI / 180.}"/>
   <!-- from ETHZ -->
-  <xacro:property name="damping_factor" default="1.5"/>
+  <xacro:property name="damping_factor" default="1.0"/>
   <xacro:property name="d0" value="${damping_factor*0.241499}"/>
   <xacro:property name="d1" value="${damping_factor*0.373279}"/>
@@ -68,19 +68,12 @@
   <xacro:property name="d5" value="${damping_factor*0.124842}"/>
   <xacro:property name="d6" value="${damping_factor*0.100000}"/>
-  <!-- <xacro:property name="d0" value="${damping_factor*0.5}"/>
-  <xacro:property name="d1" value="${damping_factor*0.5}"/>
-  <xacro:property name="d2" value="${damping_factor*0.5}"/>
-  <xacro:property name="d3" value="${damping_factor*0.5}"/>
-  <xacro:property name="d4" value="${damping_factor*0.5}"/>
-  <xacro:property name="d5" value="${damping_factor*0.5}"/>
-  <xacro:property name="d6" value="${damping_factor*0.5}"/> -->
-  <xacro:property name="friction_factor" value="1.0"/>
-  <xacro:property name="f0" value="${friction_factor*0.319088	*	1 }"/>
-  <xacro:property name="f1" value="${friction_factor*0.181301 *	1 }"/>
-  <xacro:property name="f2" value="${friction_factor*0.073019 * 1 }"/>
-  <xacro:property name="f3" value="${friction_factor*0.176713 * 1 }"/>
-  <xacro:property name="f4" value="${friction_factor*0.034631	*	1 }"/>
-  <xacro:property name="f5" value="${friction_factor*0.133913 * 1 }"/>
-  <xacro:property name="f6" value="${friction_factor*0.087096 * 1 }"/>
+  <xacro:property name="friction_factor" value="0.0"/>
+  <xacro:property name="f0" value="${friction_factor*0.319088	*	1.0 }"/>
+  <xacro:property name="f1" value="${friction_factor*0.181301}"/>
+  <xacro:property name="f2" value="${friction_factor*0.073019}"/>
+  <xacro:property name="f3" value="${friction_factor*0.176713}"/>
+  <xacro:property name="f4" value="${friction_factor*0.034631	*	1.0 }"/>
+  <xacro:property name="f5" value="${friction_factor*0.133913}"/>
+  <xacro:property name="f6" value="${friction_factor*0.087096 	*	1.0 }"/>
   <xacro:macro name="iiwa14" params="parent hardware_interface robot_name collision_postfix *origin">
     <!--joint between {parent} and link_0-->
