Commit message: revert some changes to fix sim issue

File: iiwa_description/urdf/iiwa14-master.xacro (robot description, xacro)
@@ -31,6 +31,6 @@
   <xacro:property name="safety" value="true"/>
   <!-- some constants -->
-  <xacro:property name="safety_controller_k_pos" value="100"/>
-  <xacro:property name="safety_controller_k_vel" value="10"/>
+  <xacro:property name="safety_controller_k_pos" value="50"/>
+  <xacro:property name="safety_controller_k_vel" value="2"/>
   <xacro:property name="safety_percentage" value="0.95"/>
   <xacro:property name="joint_damping" value="0.5"/>
