Commit message: relaxed max torque

File: iiwa_description/urdf/iiwa14.xacro (robot description, xacro)
@@ -32,5 +32,5 @@
   <!-- some constants -->
   <xacro:property name="safety_controller_k_pos" value="100"/>
-  <xacro:property name="safety_controller_k_vel" value="10"/>
+  <xacro:property name="safety_controller_k_vel" value="25"/>
   <xacro:property name="safety_percentage" value="0.95"/>
   <xacro:property name="joint_damping" value="0.5"/>

Commit message: increased torque limits, added print for torque limiting, added pot to center of mass of pot

File: iiwa_description/urdf/iiwa14.xacro (robot description, xacro)
@@ -32,5 +32,5 @@
   <!-- some constants -->
   <xacro:property name="safety_controller_k_pos" value="100"/>
-  <xacro:property name="safety_controller_k_vel" value="25"/>
+  <xacro:property name="safety_controller_k_vel" value="60"/>
   <xacro:property name="safety_percentage" value="0.95"/>
   <xacro:property name="joint_damping" value="0.5"/>
@@ -357,4 +357,31 @@
       </inertial>
     </link>
+<joint name="iiwa_joint_pot" type="fixed">
+      <parent link="iiwa_link_ee"/>
+      <child link="iiwa_link_pot"/>
+      <origin rpy="0 0 0" xyz="0.04 0 0.20"/>
+      <!-- <origin rpy="0 1.570796 0" xyz="0.095 0 0.15"/> -->
+    </joint>
+    <link name="iiwa_link_pot">
+      <inertial>
+        <origin rpy="0 1.57 0" xyz="0 0 0"/>
+        <mass value="0.0"/>
+        <inertia ixx="1" ixy="0" ixz="0" iyy="1" iyz="0" izz="1"/>
+      </inertial>
+      <visual>
+        <origin rpy="0 1.57 0" xyz="0 0 0"/>
+        <geometry>
+          <cylinder radius="0.1524" length="0.3556"/>
+        </geometry>
+        <material name="Grey"/>
+      </visual>
+      <collision>
+        <origin rpy="0 1.57 0" xyz="0 0 0"/>
+        <geometry>
+          <cylinder radius="0.1524" length="0.3556"/>
+        </geometry>
+        <material name="Grey"/>
+      </collision>
+    </link>
     <!--Extensions -->
     <xacro:iiwa_gazebo robot_name="${robot_name}" />

Commit message: tuned pot com

File: iiwa_description/urdf/iiwa14.xacro (robot description, xacro)
@@ -357,8 +357,9 @@
       </inertial>
     </link>
-<joint name="iiwa_joint_pot" type="fixed">
+    <joint name="iiwa_joint_pot" type="fixed">
       <parent link="iiwa_link_ee"/>
       <child link="iiwa_link_pot"/>
-      <origin rpy="0 0 0" xyz="0.04 0 0.20"/>
+      <!-- <origin rpy="0 0 0" xyz="0.015 -0.02 0.16"/> HIGHLY TUNED-->
+      <origin rpy="0 0 0" xyz="-0.01 -0.01 0.16"/>
       <!-- <origin rpy="0 1.570796 0" xyz="0.095 0 0.15"/> -->
     </joint>

Commit message: edited urdf

File: iiwa_description/urdf/iiwa14.xacro (robot description, xacro)
@@ -357,11 +357,31 @@
       </inertial>
     </link>
-    <joint name="iiwa_joint_pot" type="fixed">
+    <joint name="${robot_name}_joint_pot" type="fixed">
+    <!-- prismatic -->
       <parent link="iiwa_link_ee"/>
       <child link="iiwa_link_pot"/>
+      <origin rpy="0 0 0" xyz="0 0 0"/>
+      <axis xyz="0 0 1"/>
+      <limit lower="0" upper="1"
+             effort="100" velocity="100" />
       <!-- <origin rpy="0 0 0" xyz="0.015 -0.02 0.16"/> HIGHLY TUNED-->
-      <origin rpy="0 0 0" xyz="-0.01 -0.01 0.16"/>
+      <!-- <origin rpy="0 0 0" xyz="-0.01 -0.01 0.16"/> -->
       <!-- <origin rpy="0 1.570796 0" xyz="0.095 0 0.15"/> -->
     </joint>
+    <!-- <joint name="${robot_name}_joint_7" type="revolute">
+      <parent link="${robot_name}_link_6"/>
+      <child link="${robot_name}_link_7"/>
+      <origin xyz="0 0 0" rpy="0 0 0"/>
+      <axis xyz="0 0 1"/>
+      <limit lower="${-joint_limit_7 * PI / 180}" upper="${joint_limit_7 * PI / 180}"
+             effort="${max_effort_7}" velocity="${max_velocity_7}" />
+      <xacro:safe_controller safety="${safety}"
+                               lower="${-safety_percentage * joint_limit_7 * PI / 180}"
+                               upper="${safety_percentage * joint_limit_7 * PI / 180}"
+                               k_p="${safety_controller_k_pos}"
+                               k_v="${safety_controller_k_vel}"/>
+      <dynamics damping="${joint_damping}"/>
+    </joint>
+     -->
     <link name="iiwa_link_pot">
       <inertial>
@@ -370,5 +390,5 @@
         <inertia ixx="1" ixy="0" ixz="0" iyy="1" iyz="0" izz="1"/>
       </inertial>
-      <visual>
+      <!-- <visual>
         <origin rpy="0 1.57 0" xyz="0 0 0"/>
         <geometry>
@@ -376,5 +396,5 @@
         </geometry>
         <material name="Grey"/>
-      </visual>
+      </visual> -->
       <collision>
         <origin rpy="0 1.57 0" xyz="0 0 0"/>

Commit message: com pot tuned

File: iiwa_description/urdf/iiwa14.xacro (robot description, xacro)
@@ -361,5 +361,6 @@
       <parent link="iiwa_link_ee"/>
       <child link="iiwa_link_pot"/>
-      <origin rpy="0 0 0" xyz="0 0 0"/>
+      <origin rpy="0 0 0" xyz="0.02 0.01 0.15"/>
+      <!-- <origin rpy="0 0 0" xyz="0 0 0"/> -->
       <axis xyz="0 0 1"/>
       <limit lower="0" upper="1"
@@ -367,5 +368,4 @@
       <!-- <origin rpy="0 0 0" xyz="0.015 -0.02 0.16"/> HIGHLY TUNED-->
       <!-- <origin rpy="0 0 0" xyz="-0.01 -0.01 0.16"/> -->
-      <!-- <origin rpy="0 1.570796 0" xyz="0.095 0 0.15"/> -->
     </joint>
     <!-- <joint name="${robot_name}_joint_7" type="revolute">

Commit message: changed the inertial values - from drake

File: iiwa_description/urdf/iiwa14.xacro (robot description, xacro)
@@ -110,8 +110,8 @@
     <link name="${robot_name}_link_1">
       <inertial>
-        <origin xyz="0 -0.03 0.12" rpy="0 0 0"/>
-        <mass value="4"/>
-        <inertia ixx="0.1"  ixy="0"  ixz="0" iyy="0.09" iyz="0" izz="0.02" />
-      </inertial>
+      <origin rpy="0 0 0" xyz="0 -0.03 0.12"/>
+      <mass value="5.76"/>
+      <inertia ixx="0.033" ixy="0" ixz="0" iyy="0.0333" iyz="0" izz="0.0123"/>
+    </inertial>
       <visual>
         <origin xyz="0 0 0" rpy="0 0 0"/>
@@ -146,8 +146,10 @@
     <link name="${robot_name}_link_2">
       <inertial>
-        <origin xyz="0.0003 0.059 0.042" rpy="0 0 0"/>
-        <mass value="4"/>
-        <inertia ixx="0.05"  ixy="0"  ixz="0" iyy="0.018" iyz="0" izz="0.044" />
-      </inertial>
+      <origin rpy="0 0 0" xyz="0.0003 0.059 0.042"/>
+      <mass value="6.35"/>
+      <!-- 3.95 kuka CAD value-->
+      <!--4 Original Drake URDF value-->
+      <inertia ixx="0.0305" ixy="0" ixz="0" iyy="0.0304" iyz="0" izz="0.011"/>
+    </inertial>
       <visual>
         <origin xyz="0 0 0" rpy="0 0 0"/>
@@ -182,8 +184,10 @@
     <link name="${robot_name}_link_3">
       <inertial>
-        <origin xyz="0 0.03 0.13" rpy="0 0 0"/>
-        <mass value="3"/>
-        <inertia ixx="0.08"  ixy="0"  ixz="0" iyy="0.075" iyz="0" izz="0.01" />
-      </inertial>
+      <origin rpy="0 0 0" xyz="0 0.03 0.13"/>
+      <mass value="3.5"/>
+      <!--3.18 kuka CAD value-->
+      <!--3 Original Drake URDF value-->
+      <inertia ixx="0.025" ixy="0" ixz="0" iyy="0.0238" iyz="0" izz="0.0076"/>
+    </inertial>
       <visual>
         <origin xyz="0 0 0" rpy="0 0 0"/>
@@ -218,8 +222,10 @@
     <link name="${robot_name}_link_4">
       <inertial>
-        <origin xyz="0 0.067 0.034" rpy="0 0 0"/>
-        <mass value="2.7"/>
-        <inertia ixx="0.03"  ixy="0"  ixz="0" iyy="0.01" iyz="0" izz="0.029" />
-      </inertial>
+      <origin rpy="0 0 0" xyz="0 0.067 0.034"/>
+      <mass value="3.5"/>
+      <!--2.74 kuka CAD value-->
+      <!--2.7 Original Drake URDF value-->
+      <inertia ixx="0.017" ixy="0" ixz="0" iyy="0.0164" iyz="0" izz="0.006"/>
+    </inertial>
       <visual>
         <origin xyz="0 0 0" rpy="0 0 0"/>
@@ -254,7 +260,9 @@
     <link name="${robot_name}_link_5">
       <inertial>
-        <origin xyz="0.0001 0.021 0.076" rpy="0 0 0"/>
-        <mass value="1.7"/>
-        <inertia ixx="0.02"  ixy="0"  ixz="0" iyy="0.018" iyz="0" izz="0.005" />
+      <origin rpy="0 0 0" xyz="0.0001 0.021 0.076"/>
+      <mass value="3.5"/>
+      <!--1.69 kuka CAD value-->
+      <!--1.7 Original Drake URDF value-->
+      <inertia ixx="0.01" ixy="0" ixz="0" iyy="0.0087" iyz="0" izz="0.00449"/>
       </inertial>
       <visual>
@@ -290,8 +298,10 @@
     <link name="${robot_name}_link_6">
       <inertial>
-        <origin xyz="0 0.0006 0.0004" rpy="0 0 0"/>
-        <mass value="1.8"/>
-        <inertia ixx="0.005"  ixy="0"  ixz="0" iyy="0.0036" iyz="0" izz="0.0047" />
-      </inertial>
+      <origin rpy="0 0 0" xyz="0 0.0006 0.0004"/>
+      <mass value="1.8"/>
+      <!--1.8 kuka CAD value-->
+      <!--1.8 Original Drake URDF value-->
+      <inertia ixx="0.0049" ixy="0" ixz="0" iyy="0.0047" iyz="0" izz="0.0036"/>
+    </inertial>
       <visual>
         <origin xyz="0 0 0" rpy="0 0 0"/>
@@ -326,8 +336,10 @@
     <link name="${robot_name}_link_7">
       <inertial>
-        <origin xyz="0 0 0.02" rpy="0 0 0"/>
-        <mass value="0.3"/>
-        <inertia ixx="0.001"  ixy="0"  ixz="0" iyy="0.001" iyz="0" izz="0.001" />
-      </inertial>
+      <origin rpy="0 0 0" xyz="0 0 0.02"/>
+      <mass value="1.2"/>
+      <!--0.31 kuka CAD value-->
+      <!--0.3 Original Drake URDF value-->
+      <inertia ixx="0.001" ixy="0" ixz="0" iyy="0.001" iyz="0" izz="0.001"/>
+    </inertial>
       <visual>
         <origin xyz="0 0 0" rpy="0 0 0"/>

Commit message: added EE offset to urdf

File: iiwa_description/urdf/iiwa14.xacro (robot description, xacro)
@@ -364,5 +364,6 @@
     <link name="${robot_name}_link_ee">
       <inertial>
-        <origin xyz="0 0 0" rpy="0 0 0"/>
+        <!-- <origin xyz="0 0 0" rpy="0 0 0"/> -->
+        <origin xyz="0 0 0.155" rpy="0 0 0"/>
         <mass value="1e-6"/>
         <inertia ixx="1"  ixy="0"  ixz="0" iyy="1" iyz="0" izz="1" />

Commit message: tried gripper

File: iiwa_description/urdf/iiwa14.xacro (robot description, xacro)
@@ -361,4 +361,5 @@
       <child link="${robot_name}_link_ee"/>
       <origin xyz="0 0 0.045" rpy="0 0 0"/>
+      <!-- <origin xyz="0 0 0.25" rpy="0 0 0"/> -->
     </joint>
     <link name="${robot_name}_link_ee">
@@ -367,4 +368,5 @@
         <origin xyz="0 0 0.155" rpy="0 0 0"/>
         <mass value="1e-6"/>
+        <!-- <mass value="1.5"/> -->
         <inertia ixx="1"  ixy="0"  ixz="0" iyy="1" iyz="0" izz="1" />
       </inertial>
@@ -375,2 +377,280 @@
   </xacro:macro>
 </robot>
+    <!-- <joint name="iiwa_gripper_joint" type="fixed">
+      <parent link="iiwa_link_7"/>
+      <child link="robotiq_arg2f_base_link"/>
+      <origin rpy="0 0 0" xyz="0 0 0.045"/>
+    </joint>
+    <link name="robotiq_arg2f_base_link">
+      <inertial>
+        <origin rpy="0 0 0" xyz="8.625E-08 -4.6583E-06 0.03145"/>
+        <mass value="0.22652"/>
+        <inertia ixx="0.00020005" ixy="-4.2442E-10" ixz="-2.9069E-10" iyy="0.00017832" iyz="-3.4402E-08" izz="0.00013478"/>
+      </inertial>
+      <visual>
+        <origin rpy="0 0 0" xyz="0 0 0"/>
+        <geometry>
+          <mesh filename="package://robotiq_2f_85_gripper_visualization/meshes/visual/robotiq_arg2f_85_base_link.dae" scale="0.001 0.001 0.001"/>
+        </geometry>
+        <material name="">
+          <color rgba="0.1 0.1 0.1 1"/>
+        </material>
+      </visual>
+      <collision>
+        <origin rpy="0 0 0" xyz="0 0 0"/>
+        <geometry>
+          <mesh filename="package://robotiq_2f_85_gripper_visualization/meshes/collision/robotiq_arg2f_base_link.stl"/>
+        </geometry>
+      </collision>
+    </link>
+    <link name="left_outer_knuckle">
+      <inertial>
+          <origin xyz="-0.000200000000003065 0.0199435877845359 0.0292245259211331" rpy="0 0 0" />
+          <mass value="0.00853198276973456" />
+          <inertia ixx="2.89328108496468E-06" ixy="-1.57935047237397E-19" ixz="-1.93980378593255E-19" iyy="1.86719750325683E-06" iyz="-1.21858577871576E-06" izz="1.21905238907251E-06" />
+          </inertial>
+      <visual>
+        <origin rpy="0 0 0" xyz="0 0 0"/>
+        <geometry>
+          <mesh filename="package://robotiq_2f_85_gripper_visualization/meshes/visual/robotiq_arg2f_85_outer_knuckle.dae" scale="0.001 0.001 0.001"/>
+        </geometry>
+        <material name="">
+          <color rgba="0.792156862745098 0.819607843137255 0.933333333333333 1"/>
+        </material>
+      </visual>
+      <collision>
+        <origin rpy="0 0 0" xyz="0 0 0"/>
+        <geometry>
+          <mesh filename="package://robotiq_2f_85_gripper_visualization/meshes/collision/robotiq_arg2f_85_outer_knuckle.dae" scale="0.001 0.001 0.001"/>
+        </geometry>
+      </collision>
+    </link>
+    <link name="left_outer_finger">
+      <inertial>
+          <origin xyz="0.00030115855001899 0.0373907951953854 -0.0208027427000385" rpy="0 0 0" />
+          <mass value="0.022614240507152" />
+          <inertia ixx="1.52518312458174E-05" ixy="9.76583423954399E-10" ixz="-5.43838577022588E-10" iyy="6.17694243867776E-06" iyz="6.78636130740228E-06" izz="1.16494917907219E-05" />
+          </inertial>
+      <visual>
+        <origin rpy="0 0 0" xyz="0 0 0"/>
+        <geometry>
+          <mesh filename="package://robotiq_2f_85_gripper_visualization/meshes/visual/robotiq_arg2f_85_outer_finger.dae" scale="0.001 0.001 0.001"/>
+        </geometry>
+        <material name="">
+          <color rgba="0.1 0.1 0.1 1"/>
+        </material>
+      </visual>
+      <collision>
+        <origin rpy="0 0 0" xyz="0 0 0"/>
+        <geometry>
+          <mesh filename="package://robotiq_2f_85_gripper_visualization/meshes/collision/robotiq_arg2f_85_outer_finger.dae" scale="0.001 0.001 0.001"/>
+        </geometry>
+      </collision>
+    </link>
+    <link name="left_inner_finger">
+      <inertial>
+          <origin xyz="0.000299999999999317 0.0160078233491243 -0.0136945669206257" rpy="0 0 0" />
+          <mass value="0.0104003125914103" />
+          <inertia ixx="2.71909453810972E-06" ixy="1.35402465472579E-21" ixz="-7.1817349065269E-22" iyy="7.69100314106116E-07" iyz="6.74715432769696E-07" izz="2.30315190420171E-06" />
+          </inertial>
+      <visual>
+        <origin rpy="0 0 0" xyz="0 0 0"/>
+        <geometry>
+          <mesh filename="package://robotiq_2f_85_gripper_visualization/meshes/visual/robotiq_arg2f_85_umi.stl" scale="0.0001 0.0001 0.0001"/>
+        </geometry>
+        <material name="">
+          <color rgba="0.1 0.1 0.1 1"/>
+        </material>
+      </visual>
+      <collision>
+        <origin rpy="0 0 0" xyz="0 0 0"/>
+        <geometry>
+          <mesh filename="package://robotiq_2f_85_gripper_visualization/meshes/visual/robotiq_arg2f_85_umi.stl" scale="0.0001 0.0001 0.0001"/>
+        </geometry>
+      </collision>
+    </link>
+    <link name="left_inner_finger_pad">
+    </link>
+    <link name="left_inner_knuckle">
+      <inertial>
+          <origin xyz="0.000123011831763771 0.0507850843201817 0.00103968640075166" rpy="0 0 0" />
+        <mass value="0.0271177346495152" />
+          <inertia ixx="2.61910379223783E-05" ixy="-2.43616858946494E-07" ixz="-6.37789906117123E-09" iyy="2.8270243746167E-06" iyz="-5.37200748039765E-07" izz="2.83695868220296E-05" />
+          </inertial>
+      <visual>
+        <origin rpy="0 0 0" xyz="0 0 0"/>
+        <geometry>
+          <mesh filename="package://robotiq_2f_85_gripper_visualization/meshes/visual/robotiq_arg2f_85_inner_knuckle.dae" scale="0.001 0.001 0.001"/>
+        </geometry>
+        <material name="">
+          <color rgba="0.1 0.1 0.1 1"/>
+        </material>
+      </visual>
+      <collision>
+        <origin rpy="0 0 0" xyz="0 0 0"/>
+        <geometry>
+          <mesh filename="package://robotiq_2f_85_gripper_visualization/meshes/collision/robotiq_arg2f_85_inner_knuckle.dae" scale="0.001 0.001 0.001"/>
+        </geometry>
+      </collision>
+    </link>
+    <link name="right_outer_knuckle">
+      <inertial>
+          <origin xyz="-0.000200000000003065 0.0199435877845359 0.0292245259211331" rpy="0 0 0" />
+          <mass value="0.00853198276973456" />
+          <inertia ixx="2.89328108496468E-06" ixy="-1.57935047237397E-19" ixz="-1.93980378593255E-19" iyy="1.86719750325683E-06" iyz="-1.21858577871576E-06" izz="1.21905238907251E-06" />
+          </inertial>
+      <visual>
+        <origin rpy="0 0 0" xyz="0 0 0"/>
+        <geometry>
+          <mesh filename="package://robotiq_2f_85_gripper_visualization/meshes/visual/robotiq_arg2f_85_outer_knuckle.dae" scale="0.001 0.001 0.001"/>
+        </geometry>
+        <material name="">
+          <color rgba="0.792156862745098 0.819607843137255 0.933333333333333 1"/>
+        </material>
+      </visual>
+      <collision>
+        <origin rpy="0 0 0" xyz="0 0 0"/>
+        <geometry>
+          <mesh filename="package://robotiq_2f_85_gripper_visualization/meshes/collision/robotiq_arg2f_85_outer_knuckle.dae" scale="0.001 0.001 0.001"/>
+        </geometry>
+      </collision>
+    </link>
+    <link name="right_outer_finger">
+      <inertial>
+          <origin xyz="0.00030115855001899 0.0373907951953854 -0.0208027427000385" rpy="0 0 0" />
+          <mass value="0.022614240507152" />
+          <inertia ixx="1.52518312458174E-05" ixy="9.76583423954399E-10" ixz="-5.43838577022588E-10" iyy="6.17694243867776E-06" iyz="6.78636130740228E-06" izz="1.16494917907219E-05" />
+          </inertial>
+      <visual>
+        <origin rpy="0 0 0" xyz="0 0 0"/>
+        <geometry>
+          <mesh filename="package://robotiq_2f_85_gripper_visualization/meshes/visual/robotiq_arg2f_85_outer_finger.dae" scale="0.001 0.001 0.001"/>
+        </geometry>
+        <material name="">
+          <color rgba="0.1 0.1 0.1 1"/>
+        </material>
+      </visual>
+      <collision>
+        <origin rpy="0 0 0" xyz="0 0 0"/>
+        <geometry>
+          <mesh filename="package://robotiq_2f_85_gripper_visualization/meshes/collision/robotiq_arg2f_85_outer_finger.dae" scale="0.001 0.001 0.001"/>
+        </geometry>
+      </collision>
+    </link>
+    <link name="right_inner_finger">
+      <inertial>
+          <origin xyz="0.000299999999999317 0.0160078233491243 -0.0136945669206257" rpy="0 0 0" />
+          <mass value="0.0104003125914103" />
+          <inertia ixx="2.71909453810972E-06" ixy="1.35402465472579E-21" ixz="-7.1817349065269E-22" iyy="7.69100314106116E-07" iyz="6.74715432769696E-07" izz="2.30315190420171E-06" />
+          </inertial>
+      <visual>
+        <origin rpy="0 0 0" xyz="0 0 0"/>
+        <geometry>
+          <mesh filename="package://robotiq_2f_85_gripper_visualization/meshes/visual/robotiq_arg2f_85_umi.stl" scale="0.0001 0.0001 0.0001"/>
+        </geometry>
+        <material name="">
+          <color rgba="0.1 0.1 0.1 1"/>
+        </material>
+      </visual>
+      <collision>
+        <origin rpy="0 0 0" xyz="0 0 0"/>
+        <geometry>
+          <mesh filename="package://robotiq_2f_85_gripper_visualization/meshes/visual/robotiq_arg2f_85_umi.stl" scale="0.0001 0.0001 0.0001"/>
+        </geometry>
+      </collision>
+    </link>
+    <link name="right_inner_finger_pad">
+    </link>
+    <link name="right_inner_knuckle">
+      <inertial>
+          <origin xyz="0.000123011831763771 0.0507850843201817 0.00103968640075166" rpy="0 0 0" />
+        <mass value="0.0271177346495152" />
+          <inertia ixx="2.61910379223783E-05" ixy="-2.43616858946494E-07" ixz="-6.37789906117123E-09" iyy="2.8270243746167E-06" iyz="-5.37200748039765E-07" izz="2.83695868220296E-05" />
+          </inertial>
+      <visual>
+        <origin rpy="0 0 0" xyz="0 0 0"/>
+        <geometry>
+          <mesh filename="package://robotiq_2f_85_gripper_visualization/meshes/visual/robotiq_arg2f_85_inner_knuckle.dae" scale="0.001 0.001 0.001"/>
+        </geometry>
+        <material name="">
+          <color rgba="0.1 0.1 0.1 1"/>
+        </material>
+      </visual>
+      <collision>
+        <origin rpy="0 0 0" xyz="0 0 0"/>
+        <geometry>
+          <mesh filename="package://robotiq_2f_85_gripper_visualization/meshes/collision/robotiq_arg2f_85_inner_knuckle.dae" scale="0.001 0.001 0.001"/>
+        </geometry>
+      </collision>
+    </link>
+    <joint name="finger_joint" type="fixed">
+      <origin rpy="0 0 3.141592653589793" xyz="0 -0.0306011 0.054904"/>
+      <parent link="robotiq_arg2f_base_link"/>
+      <child link="left_outer_knuckle"/>
+      <axis xyz="1 0 0"/>
+      <limit effort="1000" lower="0" upper="0.8" velocity="2.0"/>
+    </joint>
+    <joint name="left_outer_finger_joint" type="fixed">
+      <origin rpy="0 0 0" xyz="0 0.0315 -0.0041"/>
+      <parent link="left_outer_knuckle"/>
+      <child link="left_outer_finger"/>
+      <axis xyz="1 0 0"/>
+    </joint>
+    <joint name="left_inner_knuckle_joint" type="fixed">
+      <origin rpy="0 0 3.141592653589793" xyz="0 -0.0127 0.06142"/>
+      <parent link="robotiq_arg2f_base_link"/>
+      <child link="left_inner_knuckle"/>
+      <axis xyz="1 0 0"/>
+      <limit effort="1000" lower="0" upper="0.8757" velocity="2.0"/>
+      <mimic joint="finger_joint" multiplier="1" offset="0"/>
+    </joint>
+    <joint name="left_inner_finger_joint" type="fixed">
+      <origin rpy="0 0 0" xyz="0 0.0061 0.0471"/>
+      <parent link="left_outer_finger"/>
+      <child link="left_inner_finger"/>
+      <axis xyz="1 0 0"/>
+      <limit effort="1000" lower="0" upper="0.8757" velocity="2.0"/>
+      <mimic joint="finger_joint" multiplier="-1" offset="0"/>
+    </joint>
+    <joint name="left_inner_finger_pad_joint" type="fixed">
+      <origin rpy="0 0 0" xyz="0 -0.0220203446692936 0.03242"/>
+      <parent link="left_inner_finger"/>
+      <child link="left_inner_finger_pad"/>
+      <axis xyz="0 0 1"/>
+    </joint>
+    <joint name="right_outer_knuckle_joint" type="fixed">
+      <origin rpy="0 0 0" xyz="0 0.0306011 0.054904"/>
+      <parent link="robotiq_arg2f_base_link"/>
+      <child link="right_outer_knuckle"/>
+      <axis xyz="1 0 0"/>
+      <limit effort="1000" lower="0" upper="0.81" velocity="2.0"/>
+      <mimic joint="finger_joint" multiplier="1" offset="0"/>
+    </joint>
+    <joint name="right_outer_finger_joint" type="fixed">
+      <origin rpy="0 0 0" xyz="0 0.0315 -0.0041"/>
+      <parent link="right_outer_knuckle"/>
+      <child link="right_outer_finger"/>
+      <axis xyz="1 0 0"/>
+    </joint>
+    <joint name="right_inner_knuckle_joint" type="fixed">
+      <origin rpy="0 0 0.0" xyz="0 0.0127 0.06142"/>
+      <parent link="robotiq_arg2f_base_link"/>
+      <child link="right_inner_knuckle"/>
+      <axis xyz="1 0 0"/>
+      <limit effort="1000" lower="0" upper="0.8757" velocity="2.0"/>
+      <mimic joint="finger_joint" multiplier="1" offset="0"/>
+    </joint>
+    <joint name="right_inner_finger_joint" type="fixed">
+      <origin rpy="0 0 0" xyz="0 0.0061 0.0471"/>
+      <parent link="right_outer_finger"/>
+      <child link="right_inner_finger"/>
+      <axis xyz="1 0 0"/>
+      <limit effort="1000" lower="0" upper="0.8757" velocity="2.0"/>
+      <mimic joint="finger_joint" multiplier="-1" offset="0"/>
+    </joint>
+    <joint name="right_inner_finger_pad_joint" type="fixed">
+      <origin rpy="0 0 0" xyz="0 -0.0220203446692936 0.03242"/>
+      <parent link="right_inner_finger"/>
+      <child link="right_inner_finger_pad"/>
+      <axis xyz="0 0 1"/>
+    </joint> -->
