Commit message: new urdf setting

File: iiwa_description/urdf/iiwa14.xacro (robot description, xacro)
@@ -32,5 +32,5 @@
   <!-- some constants -->
   <xacro:property name="safety_controller_k_pos" value="100"/>
-  <xacro:property name="safety_controller_k_vel" value="10"/>
+  <xacro:property name="safety_controller_k_vel" value="60"/>
   <xacro:property name="safety_percentage" value="0.95"/>
   <xacro:property name="joint_damping" value="0.5"/>
@@ -185,8 +185,10 @@
       <inertial>
       <origin rpy="0 0 0" xyz="0 0.03 0.13"/>
-      <mass value="3.5"/>
-      <!--3.18 kuka CAD value-->
-      <!--3 Original Drake URDF value-->
-      <inertia ixx="0.025" ixy="0" ixz="0" iyy="0.0238" iyz="0" izz="0.0076"/>
+      <!-- iiwa7 -->
+      <mass value="4.05623"/>
+      <inertia ixx="0.03204"  ixy="0"  ixz="0" iyy="0.00972" iyz="0.006227" izz="0.03042" />
+      <!-- DRAKE -->
+      <!-- <mass value="3.5"/> -->
+      <!-- <inertia ixx="0.025" ixy="0" ixz="0" iyy="0.0238" iyz="0" izz="0.0076"/> -->
     </inertial>
       <visual>
@@ -261,7 +263,6 @@
       <inertial>
       <origin rpy="0 0 0" xyz="0.0001 0.021 0.076"/>
+      <!--  iiwa7 -->
       <mass value="3.5"/>
-      <!--1.69 kuka CAD value-->
-      <!--1.7 Original Drake URDF value-->
       <inertia ixx="0.01" ixy="0" ixz="0" iyy="0.0087" iyz="0" izz="0.00449"/>
       </inertial>
@@ -299,8 +300,10 @@
       <inertial>
       <origin rpy="0 0 0" xyz="0 0.0006 0.0004"/>
-      <mass value="1.8"/>
-      <!--1.8 kuka CAD value-->
-      <!--1.8 Original Drake URDF value-->
-      <inertia ixx="0.0049" ixy="0" ixz="0" iyy="0.0047" iyz="0" izz="0.0036"/>
+      <!--  iiwa7 -->
+      <mass value="2.3466"/>
+      <inertia ixx="0.006509"  ixy="0"  ixz="0" iyy="0.006259" iyz="0.00031891" izz="0.004527" />
+      <!-- DRAKE -->
+      <!-- <mass value="1.8"/> -->
+      <!-- <inertia ixx="0.0049" ixy="0" ixz="0" iyy="0.0047" iyz="0" izz="0.0036"/> -->
     </inertial>
       <visual>
@@ -337,8 +340,10 @@
       <inertial>
       <origin rpy="0 0 0" xyz="0 0 0.02"/>
-      <mass value="1.2"/>
-      <!--0.31 kuka CAD value-->
-      <!--0.3 Original Drake URDF value-->
-      <inertia ixx="0.001" ixy="0" ixz="0" iyy="0.001" iyz="0" izz="0.001"/>
+      <!-- iiwa7 -->
+      <mass value="3.129"/>
+      <inertia ixx="0.01464"  ixy="0.0005912"  ixz="0" iyy="0.01465" iyz="0" izz="0.002872" />
+      <!-- DRAKE -->
+      <!-- <mass value="1.2"/> -->
+      <!-- <inertia ixx="0.001" ixy="0" ixz="0" iyy="0.001" iyz="0" izz="0.001"/> -->
     </inertial>
       <visual>
@@ -361,13 +366,29 @@
       <child link="${robot_name}_link_ee"/>
       <origin xyz="0 0 0.045" rpy="0 0 0"/>
-      <!-- <origin xyz="0 0 0.25" rpy="0 0 0"/> -->
     </joint>
     <link name="${robot_name}_link_ee">
       <inertial>
-        <!-- <origin xyz="0 0 0" rpy="0 0 0"/> -->
-        <origin xyz="0 0 0.155" rpy="0 0 0"/>
+        <origin xyz="0 0 0" rpy="0 0 0"/>
+        <!-- <origin xyz="0 0 0.155" rpy="0 0 0"/> -->
         <mass value="1e-6"/>
-        <!-- <mass value="1.5"/> -->
         <inertia ixx="1"  ixy="0"  ixz="0" iyy="1" iyz="0" izz="1" />
+      </inertial>
+    </link>
+    <joint name="${robot_name}_joint_gripper" type="fixed">
+      <parent link="${robot_name}_link_ee"/>
+      <child link="${robot_name}_link_gripper"/>
+      <origin xyz="0 0 0.125" rpy="0 0 0"/>
+      <axis xyz="0 0 1"/>
+      <!-- <limit effort="100" velocity="100"/> -->
+    </joint>
+    <link name="${robot_name}_link_gripper">
+      <inertial>
+        <!-- COM: put it along +z from the mounting plane.
+            Start with 6–8 cm; tune if gravity torque is off. -->
+        <origin xyz="0 0 0.0" rpy="0 0 0"/>
+        <!-- 2F-85 (~0.9–1.0 kg) + soft fingers (~0.1–0.3 kg) -->
+        <mass value="1.15"/>
+        <!-- Box inertia about COM using dims ~0.163 x 0.149 x 0.061 m -->
+        <inertia ixx="0.00248" ixy="0" ixz="0" iyy="0.00290" iyz="0" izz="0.00467" />
       </inertial>
     </link>

Commit message: urdf ETH

File: iiwa_description/urdf/iiwa14.xacro (robot description, xacro)
@@ -32,7 +32,7 @@
   <!-- some constants -->
   <xacro:property name="safety_controller_k_pos" value="100"/>
-  <xacro:property name="safety_controller_k_vel" value="60"/>
+  <xacro:property name="safety_controller_k_vel" value="2"/>
   <xacro:property name="safety_percentage" value="0.95"/>
-  <xacro:property name="joint_damping" value="0.5"/>
+  <!-- <xacro:property name="joint_damping" value="0.5"/> -->
   <!-- joint limits -->
   <xacro:property name="joint_limit_1" value="170"/>
@@ -59,4 +59,21 @@
   <xacro:property name="max_velocity_6" value="${135 * PI / 180.}"/>
   <xacro:property name="max_velocity_7" value="${135 * PI / 180.}"/>
+  <!-- from ETHZ -->
+  <xacro:property name="damping_factor" default="1.0"/>
+  <xacro:property name="d0" value="${damping_factor*0.241499}"/>
+  <xacro:property name="d1" value="${damping_factor*0.373279}"/>
+  <xacro:property name="d2" value="${damping_factor*0.110253}"/>
+  <xacro:property name="d3" value="${damping_factor*0.100000}"/>
+  <xacro:property name="d4" value="${damping_factor*0.100000}"/>
+  <xacro:property name="d5" value="${damping_factor*0.124842}"/>
+  <xacro:property name="d6" value="${damping_factor*0.100000}"/>
+  <xacro:property name="friction_factor" value="0.0"/>
+  <xacro:property name="f0" value="${friction_factor*0.319088	*	1.0 }"/>
+  <xacro:property name="f1" value="${friction_factor*0.181301}"/>
+  <xacro:property name="f2" value="${friction_factor*0.073019}"/>
+  <xacro:property name="f3" value="${friction_factor*0.176713}"/>
+  <xacro:property name="f4" value="${friction_factor*0.034631	*	1.0 }"/>
+  <xacro:property name="f5" value="${friction_factor*0.133913}"/>
+  <xacro:property name="f6" value="${friction_factor*0.087096 	*	1.0 }"/>
   <xacro:macro name="iiwa14" params="parent hardware_interface robot_name collision_postfix *origin">
     <!--joint between {parent} and link_0-->
@@ -106,12 +123,16 @@
                                k_p="${safety_controller_k_pos}"
                                k_v="${safety_controller_k_vel}"/>
-      <dynamics damping="${joint_damping}"/>
+      <!-- <dynamics damping="${joint_damping}"/> -->
+      <dynamics damping="${d0}" friction="${f0}"/>
     </joint>
     <link name="${robot_name}_link_1">
       <inertial>
-      <origin rpy="0 0 0" xyz="0 -0.03 0.12"/>
-      <mass value="5.76"/>
-      <inertia ixx="0.033" ixy="0" ixz="0" iyy="0.0333" iyz="0" izz="0.0123"/>
-    </inertial>
+        <origin xyz="-0.0035 0.001602 ${-0.031387+0.2025}" rpy="0 0 0"/>
+        <mass value="3.947808"/>
+        <inertia ixx="0.004554"  ixy="0"  ixz="0" iyy="0.004542" iyz="0" izz="0.000289" />
+        <!-- <origin rpy="0 0 0" xyz="0 -0.03 0.12"/> -->
+        <!-- <mass value="5.76"/> -->
+        <!-- <inertia ixx="0.033" ixy="0" ixz="0" iyy="0.0333" iyz="0" izz="0.0123"/> -->
+      </inertial>
       <visual>
         <origin xyz="0 0 0" rpy="0 0 0"/>
@@ -142,14 +163,16 @@
                                k_p="${safety_controller_k_pos}"
                                k_v="${safety_controller_k_vel}"/>
-      <dynamics damping="${joint_damping}"/>
+      <!-- <dynamics damping="${joint_damping}"/> -->
+      <dynamics damping="${d1}" friction="${f1}"/>
     </joint>
     <link name="${robot_name}_link_2">
       <inertial>
-      <origin rpy="0 0 0" xyz="0.0003 0.059 0.042"/>
-      <mass value="6.35"/>
-      <!-- 3.95 kuka CAD value-->
-      <!--4 Original Drake URDF value-->
-      <inertia ixx="0.0305" ixy="0" ixz="0" iyy="0.0304" iyz="0" izz="0.011"/>
-    </inertial>
+        <origin xyz="0.007671 0.166693 0.003551" rpy="0 0 0"/>
+        <mass value="4.502752"/>
+        <inertia ixx="0.000318"  ixy="0"  ixz="0" iyy="0.018" iyz="0" izz="0.000419" />
+        <!-- <origin rpy="0 0 0" xyz="0.0003 0.059 0.042"/> -->
+        <!-- <mass value="6.35"/> -->
+        <!-- <inertia ixx="0.0305" ixy="0" ixz="0" iyy="0.0304" iyz="0" izz="0.011"/> -->
+      </inertial>
       <visual>
         <origin xyz="0 0 0" rpy="0 0 0"/>
@@ -180,16 +203,20 @@
                                k_p="${safety_controller_k_pos}"
                                k_v="${safety_controller_k_vel}"/>
-      <dynamics damping="${joint_damping}"/>
+      <!-- <dynamics damping="${joint_damping}"/> -->
+      <dynamics damping="${d2}" friction="${f2}"/>
     </joint>
     <link name="${robot_name}_link_3">
       <inertial>
-      <origin rpy="0 0 0" xyz="0 0.03 0.13"/>
-      <!-- iiwa7 -->
-      <mass value="4.05623"/>
-      <inertia ixx="0.03204"  ixy="0"  ixz="0" iyy="0.00972" iyz="0.006227" izz="0.03042" />
-      <!-- DRAKE -->
-      <!-- <mass value="3.5"/> -->
-      <!-- <inertia ixx="0.025" ixy="0" ixz="0" iyy="0.0238" iyz="0" izz="0.0076"/> -->
-    </inertial>
+        <origin xyz="-0.002246 -0.034918 ${-0.026522+0.2155}" rpy="0 0 0"/>
+        <mass value="2.455197"/>
+        <inertia ixx="0.002233"  ixy="-0.000046"  ixz="0" iyy="0.002191" iyz="0" izz="0.000725" />
+        <!-- <origin rpy="0 0 0" xyz="0 0.03 0.13"/> -->
+        <!-- iiwa7 -->
+        <!-- <mass value="4.05623"/> -->
+        <!-- <inertia ixx="0.03204"  ixy="0"  ixz="0" iyy="0.00972" iyz="0.006227" izz="0.03042" /> -->
+        <!-- DRAKE -->
+        <!-- <mass value="3.5"/> -->
+        <!-- <inertia ixx="0.025" ixy="0" ixz="0" iyy="0.0238" iyz="0" izz="0.0076"/> -->
+      </inertial>
       <visual>
         <origin xyz="0 0 0" rpy="0 0 0"/>
@@ -220,14 +247,16 @@
                                k_p="${safety_controller_k_pos}"
                                k_v="${safety_controller_k_vel}"/>
-      <dynamics damping="${joint_damping}"/>
+      <!-- <dynamics damping="${joint_damping}"/> -->
+      <dynamics damping="${d3}" friction="${f3}"/>
     </joint>
     <link name="${robot_name}_link_4">
       <inertial>
-      <origin rpy="0 0 0" xyz="0 0.067 0.034"/>
-      <mass value="3.5"/>
-      <!--2.74 kuka CAD value-->
-      <!--2.7 Original Drake URDF value-->
-      <inertia ixx="0.017" ixy="0" ixz="0" iyy="0.0164" iyz="0" izz="0.006"/>
-    </inertial>
+        <origin xyz="0.000196 -0.052679 0.038182" rpy="0 0 0"/>
+        <mass value="2.611550"/>
+        <inertia ixx="0.038444"  ixy="0.000880"  ixz="-0.001120" iyy="0.011437" iyz="-0.001113" izz="0.049880" />
+        <!-- <origin rpy="0 0 0" xyz="0 0.067 0.034"/> -->
+        <!-- <mass value="3.5"/> -->
+        <!-- <inertia ixx="0.017" ixy="0" ixz="0" iyy="0.0164" iyz="0" izz="0.006"/> -->
+      </inertial>
       <visual>
         <origin xyz="0 0 0" rpy="0 0 0"/>
@@ -258,12 +287,16 @@
                                k_p="${safety_controller_k_pos}"
                                k_v="${safety_controller_k_vel}"/>
-      <dynamics damping="${joint_damping}"/>
+      <!-- <dynamics damping="${joint_damping}"/> -->
+      <dynamics damping="${d4}" friction="${f4}"/>
     </joint>
     <link name="${robot_name}_link_5">
       <inertial>
-      <origin rpy="0 0 0" xyz="0.0001 0.021 0.076"/>
-      <!--  iiwa7 -->
-      <mass value="3.5"/>
-      <inertia ixx="0.01" ixy="0" ixz="0" iyy="0.0087" iyz="0" izz="0.00449"/>
+        <origin xyz="0.000054 -0.002367 ${-0.211336+0.2155}" rpy="0 0 0"/>
+        <mass value="3.410009"/>
+        <inertia ixx="0.002769"  ixy="0"  ixz="0" iyy="0.002842" iyz="0" izz="0.000117" />
+        <!-- <origin rpy="0 0 0" xyz="0.0001 0.021 0.076"/> -->
+        <!--  iiwa7 -->
+        <!-- <mass value="3.5"/> -->
+        <!-- <inertia ixx="0.01" ixy="0" ixz="0" iyy="0.0087" iyz="0" izz="0.00449"/> -->
       </inertial>
       <visual>
@@ -295,16 +328,20 @@
                                k_p="${safety_controller_k_pos}"
                                k_v="${safety_controller_k_vel}"/>
-      <dynamics damping="${joint_damping}"/>
+      <!-- <dynamics damping="${joint_damping}"/> -->
+      <dynamics damping="${d5}" friction="${f5}"/>
     </joint>
     <link name="${robot_name}_link_6">
       <inertial>
-      <origin rpy="0 0 0" xyz="0 0.0006 0.0004"/>
-      <!--  iiwa7 -->
-      <mass value="2.3466"/>
-      <inertia ixx="0.006509"  ixy="0"  ixz="0" iyy="0.006259" iyz="0.00031891" izz="0.004527" />
-      <!-- DRAKE -->
-      <!-- <mass value="1.8"/> -->
-      <!-- <inertia ixx="0.0049" ixy="0" ixz="0" iyy="0.0047" iyz="0" izz="0.0036"/> -->
-    </inertial>
+        <origin xyz="0.000492 0.020190 -0.027496" rpy="0 0 0"/>
+        <mass value="3.387949"/>
+        <inertia ixx="0.000500"  ixy="0"  ixz="0" iyy="0.002809" iyz="0" izz="0.002315" />
+        <!-- <origin rpy="0 0 0" xyz="0 0.0006 0.0004"/> -->
+        <!--  iiwa7 -->
+        <!-- <mass value="2.3466"/> -->
+        <!-- <inertia ixx="0.006509"  ixy="0"  ixz="0" iyy="0.006259" iyz="0.00031891" izz="0.004527" /> -->
+        <!-- DRAKE -->
+        <!-- <mass value="1.8"/> -->
+        <!-- <inertia ixx="0.0049" ixy="0" ixz="0" iyy="0.0047" iyz="0" izz="0.0036"/> -->
+      </inertial>
       <visual>
         <origin xyz="0 0 0" rpy="0 0 0"/>
@@ -335,16 +372,20 @@
                                k_p="${safety_controller_k_pos}"
                                k_v="${safety_controller_k_vel}"/>
-      <dynamics damping="${joint_damping}"/>
+      <!-- <dynamics damping="${joint_damping}"/> -->
+      <dynamics damping="${d6}" friction="${f6}"/>
     </joint>
     <link name="${robot_name}_link_7">
       <inertial>
-      <origin rpy="0 0 0" xyz="0 0 0.02"/>
-      <!-- iiwa7 -->
-      <mass value="3.129"/>
-      <inertia ixx="0.01464"  ixy="0.0005912"  ixz="0" iyy="0.01465" iyz="0" izz="0.002872" />
-      <!-- DRAKE -->
-      <!-- <mass value="1.2"/> -->
-      <!-- <inertia ixx="0.001" ixy="0" ixz="0" iyy="0.001" iyz="0" izz="0.001"/> -->
-    </inertial>
+        <origin xyz="-0.03465 -0.023242 ${0.071377-0.081}" rpy="0 0 0"/>
+        <mass value="${0.354321 / 0.308 * 0.44}"/> <!--this is for the MFT Pneumatisch flange-->
+        <inertia ixx="0.007946"  ixy="0.000221"  ixz="0.000294" iyy="0.010889" iyz="-0.000294" izz="0.002944" />
+        <!-- <origin rpy="0 0 0" xyz="0 0 0.02"/> -->
+        <!-- iiwa7 -->
+        <!-- <mass value="3.129"/> -->
+        <!-- <inertia ixx="0.01464"  ixy="0.0005912"  ixz="0" iyy="0.01465" iyz="0" izz="0.002872" /> -->
+        <!-- DRAKE -->
+        <!-- <mass value="1.2"/> -->
+        <!-- <inertia ixx="0.001" ixy="0" ixz="0" iyy="0.001" iyz="0" izz="0.001"/> -->
+      </inertial>
       <visual>
         <origin xyz="0 0 0" rpy="0 0 0"/>
@@ -378,5 +419,5 @@
       <parent link="${robot_name}_link_ee"/>
       <child link="${robot_name}_link_gripper"/>
-      <origin xyz="0 0 0.125" rpy="0 0 0"/>
+      <origin xyz="0 0 0.12" rpy="0 0 0"/>
       <axis xyz="0 0 1"/>
       <!-- <limit effort="100" velocity="100"/> -->

Commit message: debug

File: iiwa_description/urdf/iiwa14.xacro (robot description, xacro)
@@ -377,6 +377,6 @@
     <link name="${robot_name}_link_7">
       <inertial>
-        <origin xyz="-0.03465 -0.023242 ${0.071377-0.081}" rpy="0 0 0"/>
-        <mass value="${0.354321 / 0.308 * 0.44}"/> <!--this is for the MFT Pneumatisch flange-->
+        <origin xyz="-0.03465 -0.023242 ${0.071377-0.0}" rpy="0 0 0"/>
+        <mass value="0.35432"/>
         <inertia ixx="0.007946"  ixy="0.000221"  ixz="0.000294" iyy="0.010889" iyz="-0.000294" izz="0.002944" />
         <!-- <origin rpy="0 0 0" xyz="0 0 0.02"/> -->
@@ -419,28 +419,23 @@
       <parent link="${robot_name}_link_ee"/>
       <child link="${robot_name}_link_gripper"/>
-      <origin xyz="0 0 0.12" rpy="0 0 0"/>
+      <origin xyz="0 0 0.16" rpy="0 0 0"/>
       <axis xyz="0 0 1"/>
       <!-- <limit effort="100" velocity="100"/> -->
     </joint>
     <link name="${robot_name}_link_gripper">
-      <inertial>
+      <!-- <inertial> -->
         <!-- COM: put it along +z from the mounting plane.
             Start with 6–8 cm; tune if gravity torque is off. -->
-        <origin xyz="0 0 0.0" rpy="0 0 0"/>
+        <!-- <origin xyz="0 0 0.0" rpy="0 0 0"/> -->
         <!-- 2F-85 (~0.9–1.0 kg) + soft fingers (~0.1–0.3 kg) -->
-        <mass value="1.15"/>
+        <!-- <mass value="1.15"/> -->
         <!-- Box inertia about COM using dims ~0.163 x 0.149 x 0.061 m -->
-        <inertia ixx="0.00248" ixy="0" ixz="0" iyy="0.00290" iyz="0" izz="0.00467" />
-      </inertial>
-    </link>
-    <!--Extensions -->
-    <xacro:iiwa_gazebo robot_name="${robot_name}" />
-    <xacro:iiwa_transmission hardware_interface="${hardware_interface}"/>
-  </xacro:macro>
-</robot>
-    <!-- <joint name="iiwa_gripper_joint" type="fixed">
-      <parent link="iiwa_link_7"/>
+        <!-- <inertia ixx="0.00248" ixy="0" ixz="0" iyy="0.00290" iyz="0" izz="0.00467" /> -->
+      <!-- </inertial> -->
+    </link>
+    <joint name="iiwa_gripper_joint" type="fixed">
+      <parent link="${robot_name}_link_ee"/>
       <child link="robotiq_arg2f_base_link"/>
-      <origin rpy="0 0 0" xyz="0 0 0.045"/>
+      <origin rpy="0 0 0" xyz="0 0 0"/>
     </joint>
     <link name="robotiq_arg2f_base_link">
@@ -716,3 +711,8 @@
       <child link="right_inner_finger_pad"/>
       <axis xyz="0 0 1"/>
-    </joint> -->
+    </joint>
+    <!--Extensions -->
+    <xacro:iiwa_gazebo robot_name="${robot_name}" />
+    <xacro:iiwa_transmission hardware_interface="${hardware_interface}"/>
+  </xacro:macro>
+</robot>

Commit message: sim tuned

File: iiwa_description/urdf/iiwa14.xacro (robot description, xacro)
@@ -413,5 +413,5 @@
         <!-- <origin xyz="0 0 0.155" rpy="0 0 0"/> -->
         <mass value="1e-6"/>
-        <inertia ixx="1"  ixy="0"  ixz="0" iyy="1" iyz="0" izz="1" />
+        <inertia ixx="1e-6"  ixy="0"  ixz="0" iyy="1e-6" iyz="0" izz="1e-6" />
       </inertial>
     </link>
@@ -424,15 +424,15 @@
     </joint>
     <link name="${robot_name}_link_gripper">
-      <!-- <inertial> -->
-        <!-- COM: put it along +z from the mounting plane.
-            Start with 6–8 cm; tune if gravity torque is off. -->
-        <!-- <origin xyz="0 0 0.0" rpy="0 0 0"/> -->
-        <!-- 2F-85 (~0.9–1.0 kg) + soft fingers (~0.1–0.3 kg) -->
-        <!-- <mass value="1.15"/> -->
-        <!-- Box inertia about COM using dims ~0.163 x 0.149 x 0.061 m -->
-        <!-- <inertia ixx="0.00248" ixy="0" ixz="0" iyy="0.00290" iyz="0" izz="0.00467" /> -->
-      <!-- </inertial> -->
-    </link>
-    <joint name="iiwa_gripper_joint" type="fixed">
+      <inertial>
+        <!-- CoM expressed in ${robot_name}_link_gripper frame -->
+        <origin xyz="5.3403e-08 -2.8842e-06 -1.1813481e-01" rpy="0 0 0"/>
+        <mass value="0.365848541"/>
+        <!-- Inertia about the CoM, expressed in link frame axes -->
+        <inertia
+          ixx="0.00129517580"  ixy="-0.00000261740673" ixz="-0.00000000008720478"
+          iyy="0.000340974786" iyz="-0.0000000453920893" izz="0.00108551857"/>
+      </inertial>
+    </link>
+    <!-- <joint name="iiwa_gripper_joint" type="fixed">
       <parent link="${robot_name}_link_ee"/>
       <child link="robotiq_arg2f_base_link"/>
@@ -528,4 +528,9 @@
     </link>
     <link name="left_inner_finger_pad">
+      <inertial>
+        <origin rpy="0 0 0" xyz="0 0 0"/>
+        <mass value="0.001"/>
+        <inertia ixx="1e-6" ixy="0" ixz="0" iyy="1e-6" iyz="0" izz="1e-6"/>
+      </inertial>
     </link>
     <link name="left_inner_knuckle">
@@ -618,4 +623,9 @@
     </link>
     <link name="right_inner_finger_pad">
+      <inertial>
+        <origin rpy="0 0 0" xyz="0 0 0"/>
+        <mass value="0.001"/>
+        <inertia ixx="1e-6" ixy="0" ixz="0" iyy="1e-6" iyz="0" izz="1e-6"/>
+      </inertial>
     </link>
     <link name="right_inner_knuckle">
@@ -711,5 +721,5 @@
       <child link="right_inner_finger_pad"/>
       <axis xyz="0 0 1"/>
-    </joint>
+    </joint> -->
     <!--Extensions -->
     <xacro:iiwa_gazebo robot_name="${robot_name}" />

Commit message: no gripper tuning

File: iiwa_description/urdf/iiwa14.xacro (robot description, xacro)
@@ -421,15 +421,16 @@
       <origin xyz="0 0 0.16" rpy="0 0 0"/>
       <axis xyz="0 0 1"/>
-      <!-- <limit effort="100" velocity="100"/> -->
     </joint>
     <link name="${robot_name}_link_gripper">
       <inertial>
         <!-- CoM expressed in ${robot_name}_link_gripper frame -->
-        <origin xyz="5.3403e-08 -2.8842e-06 -1.1813481e-01" rpy="0 0 0"/>
-        <mass value="0.365848541"/>
+        <!-- <origin xyz="0 0 -0.11813481" rpy="0 0 0"/>
+        <mass value="0.365848541"/> -->
+        <origin xyz="0 0 -0.05" rpy="0 0 0"/>
+        <mass value="1e-6"/>
         <!-- Inertia about the CoM, expressed in link frame axes -->
-        <inertia
-          ixx="0.00129517580"  ixy="-0.00000261740673" ixz="-0.00000000008720478"
+        <inertia ixx="0.00129517580"  ixy="0" ixz="-0.00000000008720478"
           iyy="0.000340974786" iyz="-0.0000000453920893" izz="0.00108551857"/>
+          <!-- “realistic lumped” (0.9–1.2 kg, CoM ~4–6 cm forward of the flange) -->
       </inertial>
     </link>

Commit message: effort sof limits deativated

File: iiwa_description/urdf/iiwa14.xacro (robot description, xacro)
@@ -31,5 +31,5 @@
   <xacro:property name="safety" value="true"/>
   <!-- some constants -->
-  <xacro:property name="safety_controller_k_pos" value="100"/>
+  <xacro:property name="safety_controller_k_pos" value="50"/>
   <xacro:property name="safety_controller_k_vel" value="2"/>
   <xacro:property name="safety_percentage" value="0.95"/>
