Commit message: tried ETH urdf

File: iiwa_description/urdf/iiwa14.xacro (robot description, xacro)
@@ -358,51 +358,22 @@
       </inertial>
     </link>
-    <joint name="${robot_name}_joint_pot" type="fixed">
-    <!-- prismatic -->
-      <parent link="iiwa_link_ee"/>
-      <child link="iiwa_link_pot"/>
-      <origin rpy="0 0 0" xyz="0 0 0"/>
-      <axis xyz="0 0 1"/>
-      <limit lower="0" upper="1"
-             effort="100" velocity="100" />
-      <!-- <origin rpy="0 0 0" xyz="0.015 -0.02 0.16"/> HIGHLY TUNED-->
-      <!-- <origin rpy="0 0 0" xyz="-0.01 -0.01 0.16"/> -->
-      <!-- <origin rpy="0 1.570796 0" xyz="0.095 0 0.15"/> -->
-    </joint>
-    <!-- <joint name="${robot_name}_joint_7" type="revolute">
-      <parent link="${robot_name}_link_6"/>
-      <child link="${robot_name}_link_7"/>
-      <origin xyz="0 0 0" rpy="0 0 0"/>
-      <axis xyz="0 0 1"/>
-      <limit lower="${-joint_limit_7 * PI / 180}" upper="${joint_limit_7 * PI / 180}"
-             effort="${max_effort_7}" velocity="${max_velocity_7}" />
-      <xacro:safe_controller safety="${safety}"
-                               lower="${-safety_percentage * joint_limit_7 * PI / 180}"
-                               upper="${safety_percentage * joint_limit_7 * PI / 180}"
-                               k_p="${safety_controller_k_pos}"
-                               k_v="${safety_controller_k_vel}"/>
-      <dynamics damping="${joint_damping}"/>
-    </joint>
-     -->
-    <link name="iiwa_link_pot">
-      <inertial>
-        <origin rpy="0 1.57 0" xyz="0 0 0"/>
-        <mass value="0.0"/>
-        <inertia ixx="1" ixy="0" ixz="0" iyy="1" iyz="0" izz="1"/>
-      </inertial>
-      <!-- <visual>
-        <origin rpy="0 1.57 0" xyz="0 0 0"/>
-        <geometry>
-          <cylinder radius="0.1524" length="0.3556"/>
-        </geometry>
-        <material name="Grey"/>
-      </visual> -->
-      <collision>
-        <origin rpy="0 1.57 0" xyz="0 0 0"/>
-        <geometry>
-          <cylinder radius="0.1524" length="0.3556"/>
-        </geometry>
-        <material name="Grey"/>
-      </collision>
+    <joint name="${robot_name}_joint_gripper" type="fixed">
+      <parent link="${robot_name}_link_ee"/>
+      <child link="${robot_name}_link_gripper"/>
+      <origin xyz="0 0 0.16" rpy="0 0 0"/>
+      <axis xyz="0 0 1"/>
+    </joint>
+    <link name="${robot_name}_link_gripper">
+      <inertial>
+        <!-- CoM expressed in ${robot_name}_link_gripper frame -->
+        <!-- <origin xyz="0 0 -0.11813481" rpy="0 0 0"/>
+        <mass value="0.365848541"/> -->
+        <origin xyz="0 0 -0.05" rpy="0 0 0"/>
+        <mass value="1e-6"/>
+        <!-- Inertia about the CoM, expressed in link frame axes -->
+        <inertia ixx="0.00129517580"  ixy="0" ixz="-0.00000000008720478"
+          iyy="0.000340974786" iyz="-0.0000000453920893" izz="0.00108551857"/>
+          <!-- “realistic lumped” (0.9–1.2 kg, CoM ~4–6 cm forward of the flange) -->
+      </inertial>
     </link>
     <!--Extensions -->

Commit message: added gripper

File: iiwa_description/urdf/iiwa14.xacro (robot description, xacro)
@@ -354,5 +354,24 @@
         <origin xyz="0 0 0" rpy="0 0 0"/>
         <mass value="1e-6"/>
-        <inertia ixx="1"  ixy="0"  ixz="0" iyy="1" iyz="0" izz="1" />
+        <inertia ixx="1e-6"  ixy="0"  ixz="0" iyy="1e-6" iyz="0" izz="1e-6" />
+      </inertial>
+    </link>
+    <joint name="${robot_name}_joint_gripper" type="fixed">
+      <parent link="${robot_name}_link_ee"/>
+      <child link="${robot_name}_link_gripper"/>
+      <origin xyz="0 0 0.16" rpy="0 0 0"/>
+      <axis xyz="0 0 1"/>
+    </joint>
+    <link name="${robot_name}_link_gripper">
+      <inertial>
+        <!-- CoM expressed in ${robot_name}_link_gripper frame -->
+        <!-- <origin xyz="0 0 -0.11813481" rpy="0 0 0"/>
+        <mass value="0.365848541"/> -->
+        <origin xyz="0 0 -0.05" rpy="0 0 0"/>
+        <mass value="1e-6"/>
+        <!-- Inertia about the CoM, expressed in link frame axes -->
+        <inertia ixx="0.00129517580"  ixy="0" ixz="-0.00000000008720478"
+          iyy="0.000340974786" iyz="-0.0000000453920893" izz="0.00108551857"/>
+          <!-- “realistic lumped” (0.9–1.2 kg, CoM ~4–6 cm forward of the flange) -->
       </inertial>
     </link>

Commit message: soft limits

File: iiwa_description/urdf/iiwa14.xacro (robot description, xacro)
@@ -28,11 +28,35 @@
   <!-- Include Utilities -->
   <xacro:include filename="$(find iiwa_description)/urdf/utilities.xacro" />
-  <!-- some parameters -->
+  <!-- safety parameters -->
   <xacro:property name="safety" value="true"/>
-  <!-- some constants -->
-  <xacro:property name="safety_controller_k_pos" value="100"/>
-  <xacro:property name="safety_controller_k_vel" value="10"/>
+  <xacro:property name="safety_controller_k_pos" value="50"/>
+  <xacro:property name="safety_controller_k_vel" value="2"/>
   <xacro:property name="safety_percentage" value="0.95"/>
+  <!-- joint damping -->
   <xacro:property name="joint_damping" value="0.5"/>
+    <!-- from ETHZ -->
+  <xacro:property name="damping_factor" default="1.0"/>
+  <xacro:property name="d0" value="${damping_factor*0.241499}"/>
+  <xacro:property name="d1" value="${damping_factor*0.373279}"/>
+  <xacro:property name="d2" value="${damping_factor*0.110253}"/>
+  <xacro:property name="d3" value="${damping_factor*0.100000}"/>
+  <xacro:property name="d4" value="${damping_factor*0.100000}"/>
+  <xacro:property name="d5" value="${damping_factor*0.124842}"/>
+  <xacro:property name="d6" value="${damping_factor*0.100000}"/>
+  <!-- <xacro:property name="d0" value="${damping_factor*0.5}"/>
+  <xacro:property name="d1" value="${damping_factor*0.5}"/>
+  <xacro:property name="d2" value="${damping_factor*0.5}"/>
+  <xacro:property name="d3" value="${damping_factor*0.5}"/>
+  <xacro:property name="d4" value="${damping_factor*0.5}"/>
+  <xacro:property name="d5" value="${damping_factor*0.5}"/>
+  <xacro:property name="d6" value="${damping_factor*0.5}"/> -->
+  <xacro:property name="friction_factor" value="1.0"/>
+  <xacro:property name="f0" value="${friction_factor*0.319088	*	1 }"/>
+  <xacro:property name="f1" value="${friction_factor*0.181301 *	1 }"/>
+  <xacro:property name="f2" value="${friction_factor*0.073019 * 1 }"/>
+  <xacro:property name="f3" value="${friction_factor*0.176713 * 1 }"/>
+  <xacro:property name="f4" value="${friction_factor*0.034631	*	1 }"/>
+  <xacro:property name="f5" value="${friction_factor*0.133913 * 1 }"/>
+  <xacro:property name="f6" value="${friction_factor*0.087096 * 1 }"/>
   <!-- joint limits -->
   <xacro:property name="joint_limit_1" value="170"/>
@@ -106,5 +130,6 @@
                                k_p="${safety_controller_k_pos}"
                                k_v="${safety_controller_k_vel}"/>
-      <dynamics damping="${joint_damping}"/>
+      <!-- <dynamics damping="${joint_damping}"/> -->
+      <dynamics damping="${d0}" friction="${f0}"/>
     </joint>
     <link name="${robot_name}_link_1">
@@ -142,5 +167,6 @@
                                k_p="${safety_controller_k_pos}"
                                k_v="${safety_controller_k_vel}"/>
-      <dynamics damping="${joint_damping}"/>
+      <!-- <dynamics damping="${joint_damping}"/> -->
+      <dynamics damping="${d1}" friction="${f1}"/>
     </joint>
     <link name="${robot_name}_link_2">
@@ -178,5 +204,6 @@
                                k_p="${safety_controller_k_pos}"
                                k_v="${safety_controller_k_vel}"/>
-      <dynamics damping="${joint_damping}"/>
+      <!-- <dynamics damping="${joint_damping}"/> -->
+      <dynamics damping="${d2}" friction="${f2}"/>
     </joint>
     <link name="${robot_name}_link_3">
@@ -214,5 +241,6 @@
                                k_p="${safety_controller_k_pos}"
                                k_v="${safety_controller_k_vel}"/>
-      <dynamics damping="${joint_damping}"/>
+      <!-- <dynamics damping="${joint_damping}"/> -->
+      <dynamics damping="${d3}" friction="${f3}"/>
     </joint>
     <link name="${robot_name}_link_4">
@@ -250,5 +278,6 @@
                                k_p="${safety_controller_k_pos}"
                                k_v="${safety_controller_k_vel}"/>
-      <dynamics damping="${joint_damping}"/>
+      <!-- <dynamics damping="${joint_damping}"/> -->
+      <dynamics damping="${d4}" friction="${f4}"/>
     </joint>
     <link name="${robot_name}_link_5">
@@ -286,5 +315,6 @@
                                k_p="${safety_controller_k_pos}"
                                k_v="${safety_controller_k_vel}"/>
-      <dynamics damping="${joint_damping}"/>
+      <!-- <dynamics damping="${joint_damping}"/> -->
+      <dynamics damping="${d5}" friction="${f5}"/>
     </joint>
     <link name="${robot_name}_link_6">
@@ -322,5 +352,6 @@
                                k_p="${safety_controller_k_pos}"
                                k_v="${safety_controller_k_vel}"/>
-      <dynamics damping="${joint_damping}"/>
+      <!-- <dynamics damping="${joint_damping}"/> -->
+      <dynamics damping="${d6}" friction="${f6}"/>
     </joint>
     <link name="${robot_name}_link_7">

Commit message: moved the gripper center

File: iiwa_description/urdf/iiwa14.xacro (robot description, xacro)
@@ -391,5 +391,6 @@
       <parent link="${robot_name}_link_ee"/>
       <child link="${robot_name}_link_gripper"/>
-      <origin xyz="0 0 0.16" rpy="0 0 0"/>
+      <!-- <origin xyz="0 0 0.16" rpy="0 0 0"/> -->
+      <origin xyz="0 0 0.24" rpy="0 0 0"/>
       <axis xyz="0 0 1"/>
     </joint>

Commit message: added new gripper design stl files

File: iiwa_description/urdf/iiwa14.xacro (robot description, xacro)
@@ -391,6 +391,6 @@
       <parent link="${robot_name}_link_ee"/>
       <child link="${robot_name}_link_gripper"/>
-      <!-- <origin xyz="0 0 0.16" rpy="0 0 0"/> -->
-      <origin xyz="0 0 0.22" rpy="0 0 0"/>
+      <origin xyz="0 0 0.18" rpy="0 0 0"/>
+      <!-- <origin xyz="0 0 0.22" rpy="0 0 0"/> -->
       <axis xyz="0 0 1"/>
     </joint>
@@ -402,7 +402,8 @@
         <origin xyz="0 0 -0.05" rpy="0 0 0"/>
         <mass value="1e-6"/>
+        <inertia ixx="1e-6"  ixy="0"  ixz="0" iyy="1e-6" iyz="0" izz="1e-6" />
         <!-- Inertia about the CoM, expressed in link frame axes -->
-        <inertia ixx="0.00129517580"  ixy="0" ixz="-0.00000000008720478"
-          iyy="0.000340974786" iyz="-0.0000000453920893" izz="0.00108551857"/>
+        <!-- <inertia ixx="0.00129517580"  ixy="0" ixz="-0.00000000008720478"
+          iyy="0.000340974786" iyz="-0.0000000453920893" izz="0.00108551857"/> -->
           <!-- “realistic lumped” (0.9–1.2 kg, CoM ~4–6 cm forward of the flange) -->
       </inertial>

File: iiwa_description/urdf/robotiq_2f85_umi_gripper.xacro (robot description, xacro)
@@ -93,14 +93,14 @@
         <origin rpy="0 0 0" xyz="0 0 0"/>
         <geometry>
-          <mesh filename="package://robotiq_2f_85_gripper_visualization/meshes/visual/robotiq_arg2f_85_umi2.stl" scale="0.001 0.001 0.001"/>
-        </geometry>
-        <material name="">
-          <color rgba="0.1 0.1 0.1 1"/>
-        </material>
-      </visual>
-      <collision>
-        <origin rpy="0 0 0" xyz="0 0 0"/>
-        <geometry>
-          <mesh filename="package://robotiq_2f_85_gripper_visualization/meshes/visual/robotiq_arg2f_85_umi2.stl" scale="0.001 0.001 0.001"/>
+          <mesh filename="package://robotiq_2f_85_gripper_visualization/meshes/visual/gripper_inner_finger.stl" scale="0.001 0.001 0.001"/>
+        </geometry>
+        <material name="">
+          <color rgba="0.1 0.1 0.1 1"/>
+        </material>
+      </visual>
+      <collision>
+        <origin rpy="0 0 0" xyz="0 0 0"/>
+        <geometry>
+          <mesh filename="package://robotiq_2f_85_gripper_visualization/meshes/visual/gripper_inner_finger.stl" scale="0.001 0.001 0.001"/>
         </geometry>
       </collision>
@@ -188,14 +188,14 @@
         <origin rpy="0 0 0" xyz="0 0 0"/>
         <geometry>
-          <mesh filename="package://robotiq_2f_85_gripper_visualization/meshes/visual/robotiq_arg2f_85_umi2.stl" scale="0.001 0.001 0.001"/>
-        </geometry>
-        <material name="">
-          <color rgba="0.1 0.1 0.1 1"/>
-        </material>
-      </visual>
-      <collision>
-        <origin rpy="0 0 0" xyz="0 0 0"/>
-        <geometry>
-          <mesh filename="package://robotiq_2f_85_gripper_visualization/meshes/visual/robotiq_arg2f_85_umi2.stl" scale="0.001 0.001 0.001"/>
+          <mesh filename="package://robotiq_2f_85_gripper_visualization/meshes/visual/gripper_inner_finger.stl" scale="0.001 0.001 0.001"/>
+        </geometry>
+        <material name="">
+          <color rgba="0.1 0.1 0.1 1"/>
+        </material>
+      </visual>
+      <collision>
+        <origin rpy="0 0 0" xyz="0 0 0"/>
+        <geometry>
+          <mesh filename="package://robotiq_2f_85_gripper_visualization/meshes/visual/gripper_inner_finger.stl" scale="0.001 0.001 0.001"/>
         </geometry>
       </collision>
@@ -253,5 +253,5 @@
     </joint>
     <joint name="${prefix}left_inner_finger_joint" type="fixed">
-      <origin rpy="0 0 0" xyz="0 0.0061 0.0471"/>
+      <origin rpy="0 0 1.57079632679" xyz="0 0.0061 0.0471"/>
       <parent link="${prefix}left_outer_finger"/>
       <child link="${prefix}left_inner_finger"/>
@@ -289,5 +289,5 @@
     </joint>
     <joint name="${prefix}right_inner_finger_joint" type="fixed">
-      <origin rpy="0 0 0" xyz="0 0.0061 0.0471"/>
+      <origin rpy="0 0 1.57079632679" xyz="0 0.0061 0.0471"/>
       <parent link="${prefix}right_outer_finger"/>
       <child link="${prefix}right_inner_finger"/>
