Commit message: iiwa14: restore the physical ee->gripper offset on iiwa_joint_gripper

File: iiwa_description/urdf/iiwa14.xacro (robot description, xacro)
@@ -391,21 +391,14 @@
       <parent link="${robot_name}_link_ee"/>
       <child link="${robot_name}_link_gripper"/>
-      <origin xyz="0 0 0.18" rpy="0 0 0"/>
+      <origin xyz="0 0 0.180" rpy="0 0 0"/>
       <!-- <origin xyz="0 0 0.22" rpy="0 0 0"/> -->
       <axis xyz="0 0 1"/>
     </joint>
     <link name="${robot_name}_link_gripper">
-      <inertial>
-        <!-- CoM expressed in ${robot_name}_link_gripper frame -->
-        <!-- <origin xyz="0 0 -0.11813481" rpy="0 0 0"/>
-        <mass value="0.365848541"/> -->
+      <!-- <inertial>
         <origin xyz="0 0 -0.05" rpy="0 0 0"/>
         <mass value="1e-6"/>
         <inertia ixx="1e-6"  ixy="0"  ixz="0" iyy="1e-6" iyz="0" izz="1e-6" />
-        <!-- Inertia about the CoM, expressed in link frame axes -->
-        <!-- <inertia ixx="0.00129517580"  ixy="0" ixz="-0.00000000008720478"
-          iyy="0.000340974786" iyz="-0.0000000453920893" izz="0.00108551857"/> -->
-          <!-- “realistic lumped” (0.9–1.2 kg, CoM ~4–6 cm forward of the flange) -->
-      </inertial>
+      </inertial> -->
     </link>
     <!--Extensions -->
