Commit message: updated gripper xacro

File: iiwa_description/urdf/robotiq_2f85_umi_gripper.xacro (robot description, xacro)
@@ -91,5 +91,5 @@
       </inertial>
       <visual>
-        <origin rpy="0 0 0" xyz="0 0 0"/>
+        <origin rpy="0 0 1.57079632679" xyz="0 0 0"/>
         <geometry>
           <mesh filename="package://robotiq_2f_85_gripper_visualization/meshes/visual/gripper_inner_finger.stl" scale="0.001 0.001 0.001"/>
@@ -100,5 +100,5 @@
       </visual>
       <collision>
-        <origin rpy="0 0 0" xyz="0 0 0"/>
+        <origin rpy="0 0 1.57079632679" xyz="0 0 0"/>
         <geometry>
           <mesh filename="package://robotiq_2f_85_gripper_visualization/meshes/visual/gripper_inner_finger.stl" scale="0.001 0.001 0.001"/>
@@ -186,5 +186,5 @@
       </inertial>
       <visual>
-        <origin rpy="0 0 0" xyz="0 0 0"/>
+        <origin rpy="0 0 1.57079632679" xyz="0 0 0"/>
         <geometry>
           <mesh filename="package://robotiq_2f_85_gripper_visualization/meshes/visual/gripper_inner_finger.stl" scale="0.001 0.001 0.001"/>
@@ -195,5 +195,5 @@
       </visual>
       <collision>
-        <origin rpy="0 0 0" xyz="0 0 0"/>
+        <origin rpy="0 0 1.57079632679" xyz="0 0 0"/>
         <geometry>
           <mesh filename="package://robotiq_2f_85_gripper_visualization/meshes/visual/gripper_inner_finger.stl" scale="0.001 0.001 0.001"/>
@@ -253,5 +253,5 @@
     </joint>
     <joint name="${prefix}left_inner_finger_joint" type="fixed">
-      <origin rpy="0 0 1.57079632679" xyz="0 0.0061 0.0471"/>
+      <origin rpy="0 0 0" xyz="0 0.0061 0.0471"/>
       <parent link="${prefix}left_outer_finger"/>
       <child link="${prefix}left_inner_finger"/>
@@ -289,5 +289,5 @@
     </joint>
     <joint name="${prefix}right_inner_finger_joint" type="fixed">
-      <origin rpy="0 0 1.57079632679" xyz="0 0.0061 0.0471"/>
+      <origin rpy="0 0 0" xyz="0 0.0061 0.0471"/>
       <parent link="${prefix}right_outer_finger"/>
       <child link="${prefix}right_inner_finger"/>
