Commit message: rga - hardware - needs work+

File: iiwa_description/urdf/iiwa14.urdf.xacro (robot description, xacro)
@@ -26,4 +26,6 @@
   <!--Import the lbr iiwa macro -->
   <xacro:include filename="$(find iiwa_description)/urdf/iiwa14.xacro"/>
+  <!-- Optional UMI gripper macro -->
+  <xacro:include filename="$(find iiwa_description)/urdf/robotiq_2f85_umi_gripper.xacro"/>
   <xacro:arg name="hardware_interface" default="PositionJointInterface"/>
   <xacro:arg name="robot_name" default="iiwa"/>
@@ -31,4 +33,6 @@
   <xacro:arg name="origin_rpy" default="0 0 0"/>
   <xacro:arg name="simple_collision" default="false"/>
+  <!-- Toggle to show/hide the Robotiq UMI gripper in the URDF -->
+  <xacro:arg name="with_gripper" default="true"/>
   <!-- collision shapes -->
   <xacro:if value="$(arg simple_collision)">
@@ -44,3 +48,7 @@
     <origin xyz="$(arg origin_xyz)" rpy="$(arg origin_rpy)" />
   </xacro:iiwa14>
+  <!-- Optional gripper attachment -->
+  <xacro:if value="$(arg with_gripper)">
+    <xacro:robotiq_2f85_umi_gripper parent="$(arg robot_name)_link_ee" robot_name="$(arg robot_name)"/>
+  </xacro:if>
 </robot>

File: iiwa_description/urdf/iiwa14.xacro (robot description, xacro)
@@ -392,5 +392,5 @@
       <child link="${robot_name}_link_gripper"/>
       <!-- <origin xyz="0 0 0.16" rpy="0 0 0"/> -->
-      <origin xyz="0 0 0.24" rpy="0 0 0"/>
+      <origin xyz="0 0 0.22" rpy="0 0 0"/>
       <axis xyz="0 0 1"/>
     </joint>

Commit message: added taxels to the iiiwa14 urdf

File: iiwa_description/urdf/iiwa14.urdf.xacro (robot description, xacro)
@@ -28,4 +28,6 @@
   <!-- Optional UMI gripper macro -->
   <xacro:include filename="$(find iiwa_description)/urdf/robotiq_2f85_umi_gripper.xacro"/>
+  <!-- Optional Xela-instrumented finger assemblies -->
+  <xacro:include filename="$(find iiwa_description)/urdf/finger_with_xela.xacro"/>
   <xacro:arg name="hardware_interface" default="PositionJointInterface"/>
   <xacro:arg name="robot_name" default="iiwa"/>
@@ -35,4 +37,6 @@
   <!-- Toggle to show/hide the Robotiq UMI gripper in the URDF -->
   <xacro:arg name="with_gripper" default="true"/>
+  <!-- Toggle to attach Xela finger assemblies (requires with_gripper:=true) -->
+  <xacro:arg name="with_fingers" default="true"/>
   <!-- collision shapes -->
   <xacro:if value="$(arg simple_collision)">
@@ -51,4 +55,9 @@
   <xacro:if value="$(arg with_gripper)">
     <xacro:robotiq_2f85_umi_gripper parent="$(arg robot_name)_link_ee" robot_name="$(arg robot_name)"/>
+    <!-- Optional Xela finger assemblies (left + right) -->
+    <xacro:if value="$(arg with_fingers)">
+      <xacro:xela_finger prefix="left_finger_"  parent="left_inner_finger"/>
+      <xacro:xela_finger prefix="right_finger_" parent="right_inner_finger"/>
+    </xacro:if>
   </xacro:if>
 </robot>

File: iiwa_description/urdf/robotiq_2f85_umi_gripper.xacro (robot description, xacro)
@@ -85,5 +85,5 @@
     </link>
     <link name="${prefix}left_inner_finger">
-      <inertial>
+      <!-- <inertial>
         <origin xyz="0.000299999999999317 0.0160078233491243 -0.0136945669206257" rpy="0 0 0"/>
         <mass value="0.0104003125914103"/>
@@ -104,5 +104,5 @@
           <mesh filename="package://robotiq_2f_85_gripper_visualization/meshes/visual/gripper_inner_finger.stl" scale="0.001 0.001 0.001"/>
         </geometry>
-      </collision>
+      </collision> -->
     </link>
     <link name="${prefix}left_inner_finger_pad">
@@ -180,5 +180,5 @@
     </link>
     <link name="${prefix}right_inner_finger">
-      <inertial>
+      <!-- <inertial>
         <origin xyz="0.000299999999999317 0.0160078233491243 -0.0136945669206257" rpy="0 0 0"/>
         <mass value="0.0104003125914103"/>
@@ -199,5 +199,5 @@
           <mesh filename="package://robotiq_2f_85_gripper_visualization/meshes/visual/gripper_inner_finger.stl" scale="0.001 0.001 0.001"/>
         </geometry>
-      </collision>
+      </collision> -->
     </link>
     <link name="${prefix}right_inner_finger_pad">
